File: TeensyMaestro Main PCB/TeensyMaestro Main PCB.kicad_sch (KiCad schematic)
At the start: 6 parts

Commit message: Updated documentation in schematic
Parts:
- H1, H2, H3, H4, H5, H6: now left out of the parts list
Changed lines of the file:
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@@
 	(title_block
 		(title "KD0RC TeensyMaestro")
-		(date "2025-07-27")
-		(rev "v3.0")
+		(date "2025-09-09")
+		(rev "v3.1")
 		(company "NV0E")
 		(comment 1 "Based on original design by KD0RC.")
@@
 		(unit 1)
 		(exclude_from_sim no)
-		(in_bom yes)
+		(in_bom no)
 		(on_board yes)
 		(dnp no)
@@
 		(unit 1)
 		(exclude_from_sim no)
-		(in_bom yes)
+		(in_bom no)
 		(on_board yes)
 		(dnp no)
@@
 		(unit 1)
 		(exclude_from_sim no)
-		(in_bom yes)
+		(in_bom no)
 		(on_board yes)
 		(dnp no)
@@
 		(unit 1)
 		(exclude_from_sim no)
-		(in_bom yes)
+		(in_bom no)
 		(on_board yes)
 		(dnp no)
@@
 		(unit 1)
 		(exclude_from_sim no)
-		(in_bom yes)
+		(in_bom no)
 		(on_board yes)
 		(dnp no)
@@
 		(unit 1)
 		(exclude_from_sim no)
-		(in_bom yes)
+		(in_bom no)
 		(on_board yes)
 		(dnp no)
