File: TeensyMaestro Main PCB/TeensyMaestro Main PCB.kicad_pcb (KiCad board)
At the start: 2 copper layers, 197.3 x 121.2 mm, 115 parts, among them J16 B2B-XH-A_LF__SN_, J17 B2B-XH-A_LF__SN_, J18 B2B-XH-A_LF__SN_, J19 B2B-XH-A_LF__SN_, J2 B5B-XH-A_LF__SN_, J20 B2B-XH-A_LF__SN_, J21 B2B-XH-A_LF__SN_, J22 B3B-XH-A_LF__SN_, J26 B2B-XH-A_LF__SN_, J27 B2B-XH-A_LF__SN_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

Commit message: Updated documentation in schematic
Parts:
- SW10, SW5: value AGC-T/RIT_Sel A -> PEC11L-4120F-S0020
- SW11: value CW_Mic/Menu Sel -> PEC11L-4120F-S0020
- SW2: value RotaryEncoder_Switch_MP -> PEC11L-4120F-S0020
- SW3: value LowShift/NB A -> PEC11L-4120F-S0020
- SW4: value HighWidth/NR A -> PEC11L-4120F-S0020
- SW7: value Vol/Mute B -> PEC11L-4120F-S0020
- SW8: value LowShift/NB B -> PEC11L-4120F-S0020
- SW9: value HighWidth/NR B -> PEC11L-4120F-S0020
Changed lines of the file:
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@@
 			)
 		)
-		(property "Value" "HighWidth/NR B"
+		(property "Value" "PEC11L-4120F-S0020"
 			(at 2.5 7.45 0)
 			(layer "F.SilkS")
@@
 			)
 		)
+		(property "Purpose" "HighWidth/NR B"
+			(at 0 0 0)
+			(unlocked yes)
+			(layer "F.Fab")
+			(hide yes)
+			(effects
+				(font
+					(size 1 1)
+					(thickness 0.15)
+				)
+			)
+		)
 		(property ki_fp_filters "RotaryEncoder*Switch*")
 		(sheetname "/IO Expander B/")
@@
 		(sheetname "/")
 		(sheetfile "TeensyMaestro Main PCB.kicad_sch")
-		(attr exclude_from_pos_files)
+		(attr exclude_from_pos_files exclude_from_bom)
 		(fp_circle
 			(center 0 0)
@@
 			)
 		)
-		(property "Value" "LowShift/NB B"
+		(property "Value" "PEC11L-4120F-S0020"
 			(at 2.5 7.45 0)
 			(layer "F.SilkS")
@@
 			)
 		)
+		(property "Purpose" "LowShift/NB B"
+			(at 0 0 0)
+			(unlocked yes)
+			(layer "F.Fab")
+			(hide yes)
+			(effects
+				(font
+					(size 1 1)
+					(thickness 0.15)
+				)
+			)
+		)
 		(property ki_fp_filters "RotaryEncoder*Switch*")
 		(sheetname "/IO Expander B/")
@@
 			)
 		)
-		(property "Value" "AGC-T/RIT_Sel A"
+		(property "Value" "PEC11L-4120F-S0020"
 			(at 2.5 7.45 0)
 			(layer "F.SilkS")
@@
 			)
 		)
+		(property "Purpose" "AGC-T/RIT_Sel A"
+			(at 0 0 0)
+			(unlocked yes)
+			(layer "F.Fab")
+			(hide yes)
+			(effects
+				(font
+					(size 1 1)
+					(thickness 0.15)
+				)
+			)
+		)
 		(property ki_fp_filters "RotaryEncoder*Switch*")
 		(sheetname "/IO Expander B/")
@@
 		(sheetname "/")
 		(sheetfile "TeensyMaestro Main PCB.kicad_sch")
-		(attr exclude_from_pos_files)
+		(attr exclude_from_pos_files exclude_from_bom)
 		(fp_circle
 			(center 0 0)
@@
 		(sheetname "/")
 		(sheetfile "TeensyMaestro Main PCB.kicad_sch")
-		(attr exclude_from_pos_files)
+		(attr exclude_from_pos_files exclude_from_bom)
 		(fp_circle
 			(center 0 0)
@@
 			)
 		)
-		(property "Value" "HighWidth/NR A"
+		(property "Value" "PEC11L-4120F-S0020"
 			(at 2.5 7.45 0)
 			(layer "F.SilkS")
@@
 			)
 		)
+		(property "Purpose" "HighWidth/NR A"
+			(at 0 0 0)
+			(unlocked yes)
+			(layer "F.Fab")
+			(hide yes)
+			(effects
+				(font
+					(size 1 1)
+					(thickness 0.15)
+				)
+			)
+		)
 		(property ki_fp_filters "RotaryEncoder*Switch*")
 		(sheetname "/IO Expander A/")
@@
 			)
 		)
-		(property "Value" "RotaryEncoder_Switch_MP"
+		(property "Value" "PEC11L-4120F-S0020"
 			(at 2.5 7.45 0)
 			(layer "F.SilkS")
@@
 			)
 		)
-		(property "Value" "Vol/Mute B"
+		(property "Value" "PEC11L-4120F-S0020"
 			(at 2.5 7.45 0)
 			(layer "F.SilkS")
@@
 			)
 		)
+		(property "Purpose" "Vol/Mute B"
+			(at 0 0 0)
+			(unlocked yes)
+			(layer "F.Fab")
+			(hide yes)
+			(effects
+				(font
+					(size 1 1)
+					(thickness 0.15)
+				)
+			)
+		)
 		(property ki_fp_filters "RotaryEncoder*Switch*")
 		(sheetname "/IO Expander B/")
@@
 			)
 		)
-		(property "Value" "AGC-T/RIT_Sel A"
+		(property "Value" "PEC11L-4120F-S0020"
 			(at 2.5 7.45 0)
 			(layer "F.SilkS")
@@
 			)
 		)
+		(property "Purpose" "AGC-T/RIT_Sel A"
+			(at 0 0 0)
+			(unlocked yes)
+			(layer "F.Fab")
+			(hide yes)
+			(effects
+				(font
+					(size 1 1)
+					(thickness 0.15)
+				)
+			)
+		)
 		(property ki_fp_filters "RotaryEncoder*Switch*")
 		(sheetname "/IO Expander A/")
@@
 		(sheetname "/")
 		(sheetfile "TeensyMaestro Main PCB.kicad_sch")
-		(attr exclude_from_pos_files)
+		(attr exclude_from_pos_files exclude_from_bom)
 		(fp_circle
 			(center 0 0)
@@
 		(sheetname "/")
 		(sheetfile "TeensyMaestro Main PCB.kicad_sch")
-		(attr exclude_from_pos_files)
+		(attr exclude_from_pos_files exclude_from_bom)
 		(fp_circle
 			(center 0 0)
@@
 			)
 		)
-		(property "Value" "LowShift/NB A"
+		(property "Value" "PEC11L-4120F-S0020"
 			(at 2.5 7.45 0)
 			(layer "F.SilkS")
@@
 			)
 		)
+		(property "Purpose" "LowShift/NB A"
+			(at 0 0 0)
+			(unlocked yes)
+			(layer "F.Fab")
+			(hide yes)
+			(effects
+				(font
+					(size 1 1)
+					(thickness 0.15)
+				)
+			)
+		)
 		(property ki_fp_filters "RotaryEncoder*Switch*")
 		(sheetname "/IO Expander A/")
@@
 		(sheetname "/")
 		(sheetfile "TeensyMaestro Main PCB.kicad_sch")
-		(attr exclude_from_pos_files)
+		(attr exclude_from_pos_files exclude_from_bom)
 		(fp_circle
 			(center 0 0)
@@
 			)
 		)
-		(property "Value" "CW_Mic/Menu Sel"
+		(property "Value" "PEC11L-4120F-S0020"
 			(at 2.5 7.45 0)
 			(layer "F.SilkS")
@@
 			)
 		)
+		(property "Purpose" "CW_Mic/Menu Sel"
+			(at 0 0 0)
+			(unlocked yes)
+			(layer "F.Fab")
+			(hide yes)
+			(effects
+				(font
+					(size 1 1)
+					(thickness 0.15)
+				)
+			)
+		)
 		(property ki_fp_filters "RotaryEncoder*Switch*")
 		(sheetname "/Microcontroller/")
@@
 		(sheetname "/Microcontroller/")
 		(sheetfile "microcontroller.kicad_sch")
-		(attr through_hole)
+		(attr through_hole exclude_from_bom)
 		(fp_circle
 			(center 0 0)
@@
 		(sheetname "/Microcontroller/")
 		(sheetfile "microcontroller.kicad_sch")
-		(attr through_hole)
+		(attr through_hole exclude_from_bom)
 		(fp_circle
 			(center 0 0)
@@
 		(sheetname "/Microcontroller/")
 		(sheetfile "microcontroller.kicad_sch")
-		(attr through_hole)
+		(attr through_hole exclude_from_bom)
 		(fp_circle
 			(center 0 0)

Commit message: Update schematic & BOM with 5v pullup correction
Parts:
- C10, C25, C26, C9: value 100nF -> 1nF
Changed lines of the file:
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@@
 		(sheetname "/IO Expander B/")
 		(sheetfile "io_expander_b.kicad_sch")
-		(attr through_hole)
+		(attr through_hole exclude_from_bom dnp)
 		(fp_line
 			(start 1.04 0)
@@
 			)
 		)
-		(property "Value" "100nF"
+		(property "Value" "1nF"
 			(at 2.5 -2.5 90)
 			(layer "B.Fab")
@@
 		(sheetname "/IO Expander A/")
 		(sheetfile "io_expander_a.kicad_sch")
-		(attr through_hole)
+		(attr through_hole exclude_from_bom dnp)
 		(fp_line
 			(start 1.04 0)
@@
 		(sheetname "/IO Expander A/")
 		(sheetfile "io_expander_a.kicad_sch")
-		(attr through_hole)
+		(attr through_hole exclude_from_bom dnp)
 		(fp_line
 			(start 1.04 0)
@@
 			)
 		)
-		(property "Value" "100nF"
+		(property "Value" "1nF"
 			(at 2.5 -2.5 90)
 			(layer "B.Fab")
@@
 			)
 		)
-		(property "Value" "100nF"
+		(property "Value" "1nF"
 			(at 2.5 -2.5 90)
 			(layer "B.Fab")
@@
 		(sheetname "/IO Expander B/")
 		(sheetfile "io_expander_b.kicad_sch")
-		(attr through_hole)
+		(attr through_hole exclude_from_bom dnp)
 		(fp_line
 			(start 1.04 0)
@@
 			)
 		)
-		(property "Value" "100nF"
+		(property "Value" "1nF"
 			(at 2.5 -2.5 90)
 			(layer "B.Fab")
